File: KiCad/BB3plus CM5 STM32H7 module.kicad_pcb (KiCad board)
At the start: 6 copper layers, 55 x 40 mm, 146 parts, among them IC1 AZ1117CH2-3.3TRG1, IC10 TS3DV642A0RUAR, IC11 LSF0204GU12, IC12 MX25UM25645GXDI00-T, IC2 PI3USB102ZLEX, IC3 SN74LVC1G14DBVR, IC4 STM32H7R7L8H6H, IC5 TLV75718PDRVR, IC6 IS21EF04GP-JQLI, IC7 LAN8742A-CZ-TR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

Commit message: #14
Connections:
- IC6 pad M7: +1V8 -> GND
Routing:
- net +1V8: track 35.8 -> 35.4 mm, vias 35 -> 34
- net GND: vias 246 -> 247
Other:
- board text added: "EEZ CM5 MCU (04/2026 ${project_version})"
- board text removed: "EEZ CM5 MCU (01/2026 ${project_version})"
Changed lines of the file:
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@@
 	(title_block
 		(title "${project_name}")
-		(date "2026-01-28")
+		(date "2026-03-26")
 		(rev "${project_version}")
 		(company "${project_creator}")
@@
 	(property "project_name" "EEZ BB3+ STM32H7 CM5 module")
 	(property "project_url" "https://www.envox.eu")
-	(property "project_version" "r1B3")
+	(property "project_version" "r1B4")
 	(net 0 "")
 	(net 1 "/STM32H7 MCU/RCC_OSC_IN")
@@
 			(size 0.4064 0.4064)
 			(layers "F.Cu" "F.Mask" "F.Paste")
-			(net 121 "+1V8")
+			(net 3 "GND")
 			(pinfunction "VCCQ")
 			(pintype "power_in")
@@
 			(layer "F.Cu")
 		)
+		(fp_poly
+			(pts
+				(xy 0.3352 0.2667) (xy -0.3252 0.2667) (xy -0.3252 -0.2667) (xy 0.3352 -0.2667)
+			)
+			(stroke
+				(width 0)
+				(type solid)
+			)
+			(fill yes)
+			(layer "F.Mask")
+		)
 		(fp_rect
 			(start -2.929 -0.635)
@@
 			(layer "F.SilkS")
 		)
+		(fp_poly
+			(pts
+				(xy 0.3352 0.2667) (xy -0.3252 0.2667) (xy -0.3252 -0.2667) (xy 0.3352 -0.2667)
+			)
+			(stroke
+				(width 0)
+				(type solid)
+			)
+			(fill yes)
+			(layer "F.Paste")
+		)
 		(fp_rect
 			(start -2.929 -0.635)
@@
 		(layer "B.SilkS")
 	)
-	(gr_text "EEZ CM5 MCU (01/2026 ${project_version})"
+	(gr_text "EEZ CM5 MCU (04/2026 ${project_version})"
 		(at 119.17 109.86 0)
 		(layer "F.SilkS")
@@
 	)
 	(via
+		(at 103.37 92.853783)
+		(size 0.42)
+		(drill 0.2)
+		(layers "F.Cu" "B.Cu")
+		(net 3)
+	)
+	(via
 		(at 135.21 93.8551)
 		(size 0.42)
@@
 	)
 	(segment
-		(start 103.37 92.53)
-		(end 103.37 92.86)
-		(width 0.2032)
-		(layer "F.Cu")
-		(net 121)
-	)
-	(segment
 		(start 112.81 79.4)
 		(end 110.57 81.64)
@@
 		(size 0.42)
 		(drill 0.2)
-		(layers "F.Cu" "B.Cu")
-		(net 121)
-	)
-	(via
-		(at 103.37 92.86)
-		(size 0.42)
-		(drill 0.2)

Commit message: #15
Connections:
- IC2 pad 6: /CM5 socket/USB3_1- -> /CM5 socket/USB3_1_D-
- IC2 pad 7: /CM5 socket/USB3_1+ -> /CM5 socket/USB3_1_D+
- SoM1 pad 163: unconnected-(SoM1B-USB3-1-DP-Pad163) -> /CM5 socket/USB3_1_D+
- SoM1 pad 165: unconnected-(SoM1B-USB3-1-DM-Pad165) -> /CM5 socket/USB3_1_D-
- SoM1 pad 169: /CM5 socket/USB3_1- -> unconnected-(SoM1B-USB3-1-TX_N-Pad169)
- SoM1 pad 171: /CM5 socket/USB3_1+ -> unconnected-(SoM1B-USB3-1-TX_P-Pad171)
Routing:
- net /CM5 socket/USB3_1-: track 13.8 -> 0.00 mm, vias 1 -> 0
- net /CM5 socket/USB3_1+: track 13.7 -> 0.00 mm, vias 1 -> 0
- net /CM5 socket/USB3_1_D+: track 0.00 -> 12.6 mm, vias 0 -> 1
- net /CM5 socket/USB3_1_D-: track 0.00 -> 12.4 mm, vias 0 -> 1
