File: KiCad/BB3plus CM5 STM32H7 module.kicad_pcb (KiCad board)
At the start: 6 copper layers, 55 x 40 mm, 158 parts, among them IC1 AZ1117CH2-3.3TRG1, IC10 LSF0204GU12, IC11 MX25UM25645GXDI00-T, IC2 AZ1117CH-1.8TRG1, IC3 PI3USB102ZLEX, IC4 SN74LVC1G14DBVR, IC5 STM32H7R7L8H6H, IC6 LAN8742A-CZ-TR, IC7 APS256XXN-OBR-BG, IC8 TFP410PAP, IC9 TS3DV642A0RUAR, X1 DF40C-100DP-0.4V(51), X2 DF40C-100DP-0.4V(51), X4 5033981892, Y1 VXM7-9032-25M0000000, Y2 VXM7-9032-25M0000000

Commit message: Rename USB_FS_SEL to USB_HS_SEL
Connections:
- net USB_FS_SEL renamed USB_HS_SEL

Commit message: #20
Parts:
- added JP1: ~, PCM_EEZ_SMD:JP3 shorted (0603), B.Cu at (110.7, 77.0)
- added R1: 10K, PCM_EEZ_passives:R_0402_1005Metric, F.Cu at (112.2, 74.8)
- renumbered JP1 to JP2, JP2 to JP3, JP3 to JP4, JP4 to JP5, JP5 to JP6, JP6 to JP7, JP7 to JP8, R9 to R10, R10 to R11, R11 to R12, R12 to R13, R13 to R14, R14 to R15, R15 to R16, R16 to R17, R17 to R18, R18 to R19, R1 to R2, R19 to R20, R20 to R21, R21 to R22, R22 to R23, R23 to R24, R24 to R25, R25 to R26, R26 to R27, R27 to R28, R28 to R29, R2 to R3, R29 to R30, R30 to R31, R31 to R32, R32 to R33, R33 to R34, R34 to R35, R35 to R36, R36 to R37, R3 to R4, R4 to R5, R5 to R6, R6 to R7, R7 to R8, R8 to R9
Routing:
- net Net-(JP1-PadCOM): track 0.00 -> 2.19 mm, vias 0 -> 1
- net USB_HS_SEL: track 19.0 -> 21.1 mm
- net GND: track 116.4 -> 117.0 mm, vias 253 -> 254
- net +3V3: track 58.0 -> 58.7 mm, vias 52 -> 53
