File: KiCad/BB3plus CM5 STM32H7 module.kicad_sch (KiCad schematic)
At the start: 9 parts

Commit message: #16
Parts:
- renumbered LOGO5 to LOGO1, LOGO1 to LOGO2, LOGO2 to LOGO3, LOGO3 to LOGO4, LOGO4 to LOGO5
Changed lines of the file:
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@@
 		(dnp no)
 		(fields_autoplaced yes)
-		(property "Reference" "LOGO5"
+		(property "Reference" "LOGO1"
 			(at 60.96 195.7784 0)
 			(effects
@@
 			(project "BB3plus CM5 STM32H7 module"
 				(path "/1a4f0aea-3a69-423f-8790-3103cd0321c4"
-					(reference "LOGO5")
+					(reference "LOGO1")
 					(unit 1)
 				)
@@
 		(dnp no)
 		(fields_autoplaced yes)
-		(property "Reference" "LOGO3"
+		(property "Reference" "LOGO4"
 			(at 38.1 184.3355 0)
 			(effects
@@
 			(project "BB3plus CM5 STM32H7 module"
 				(path "/1a4f0aea-3a69-423f-8790-3103cd0321c4"
-					(reference "LOGO3")
+					(reference "LOGO4")
 					(unit 1)
 				)
@@
 		(dnp no)
 		(fields_autoplaced yes)
-		(property "Reference" "LOGO4"
+		(property "Reference" "LOGO5"
 			(at 45.72 185.964 0)
 			(effects
@@
 			(project "BB3plus CM5 STM32H7 module"
 				(path "/1a4f0aea-3a69-423f-8790-3103cd0321c4"
-					(reference "LOGO4")
+					(reference "LOGO5")
 					(unit 1)
 				)
@@
 		(dnp no)
 		(fields_autoplaced yes)
-		(property "Reference" "LOGO1"
+		(property "Reference" "LOGO2"
 			(at 22.86 185.6184 0)
 			(effects
@@
 			(project "BB3plus CM5 STM32H7 module"
 				(path "/1a4f0aea-3a69-423f-8790-3103cd0321c4"
-					(reference "LOGO1")
+					(reference "LOGO2")
 					(unit 1)
 				)
@@
 		(dnp no)
 		(fields_autoplaced yes)
-		(property "Reference" "LOGO2"
+		(property "Reference" "LOGO3"
 			(at 30.48 185.6122 0)
 			(effects
@@
 			(project "BB3plus CM5 STM32H7 module"
 				(path "/1a4f0aea-3a69-423f-8790-3103cd0321c4"
-					(reference "LOGO2")
-					(unit 1)
-				)
+					(reference "LOGO3")
+					(unit 1)
+				)

Commit message: #19
Other:
- sheet Ethernet PHY, PSRAM, eMMC renamed Ethernet PHY, PSRAM, SDcard
Changed lines of the file:
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@@
 	(title_block
 		(title "${project_name}")
-		(date "2026-04-04")
+		(date "2026-04-09")
 		(rev "${project_version}")
 		(company "${project_creator}")
@@
 			(color 0 0 0 0.0000)
 		)
-		(property "Sheetname" "Ethernet PHY, PSRAM, eMMC"
+		(property "Sheetname" "Ethernet PHY, PSRAM, SDcard"
 			(at 25.4 39.9284 0)
 			(effects

Commit message: .step file update, migration to KiCad 10
Parts:
- FM1, FM2, FM3, FM4: value ~ -> (none)
