File: KiCad/Ethernet_flash.kicad_sch (KiCad schematic)
At the start: 36 parts, among them IC10 TS3DV642A0RUAR, IC11 LSF0204GU12, IC12 MX25UM25645GXDI00-T, IC9 TFP410PAP

Commit message: #13
Parts:
- renumbered JP1 to JP2
Connections:
- net DVID_SEL1 is gone; now on net +3V3: IC10.16 (SEL1)
- net ~{RESET_OUT}: no longer IC10.2 (EN)
- net DVID_SEL2 renamed VMUX_SEL
- new net VMUX_EN: IC10.2 (EN)

Commit message: #14
Other:
- note added: "Connect?"
- note added: "Consumption (VCC Read), 200 MHz 8IO DTR (SIO floating): Typ. 55 mA, Max. 80 mA"
- note added: "Pulldown?"
Changed lines of the file:
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@@
 	(title_block
 		(title "${project_name}")
-		(date "2026-01-29")
+		(date "2026-03-26")
 		(rev "${project_version}")
 		(company "${project_creator}")
@@
 		(comment 2 "${project_info}")
 		(comment 3 "${project_url}")
+	)
+	(rectangle
+		(start 161.925 108.585)
+		(end 172.085 133.985)
+		(stroke
+			(width 0)
+			(type solid)
+			(color 255 0 0 1)
+		)
+		(fill
+			(type none)
+		)
+	)
+	(rectangle
+		(start 64.135 87.63)
+		(end 88.265 94.615)
+		(stroke
+			(width 0)
+			(type solid)
+			(color 255 0 0 1)
+		)
+		(fill
+			(type none)
+		)
 	)
 	(text "RGB-to-DVID converter"
@@
 		)
 	)
+	(text "Pulldown?"
+		(exclude_from_sim no)
+		(at 166.37 133.35 0)
+		(effects
+			(font
+				(size 0.889 0.889)
+				(color 255 0 0 1)
+			)
+		)
+	)
 	(text "Video MUX 1:2"
 		(exclude_from_sim no)
@@
 		)
 	)
+	(text "Consumption (VCC Read), 200 MHz 8IO DTR (SIO floating): Typ. 55 mA, Max. 80 mA"
+		(exclude_from_sim no)
+		(at 187.96 86.36 0)
+		(effects
+			(font
+				(size 0.889 0.889)
+				(color 132 0 132 1)
+			)
+			(justify left bottom)
+		)
+	)
+	(text "Connect?"
+		(exclude_from_sim no)
+		(at 103.505 93.98 0)
+		(effects
+			(font
+				(size 0.889 0.889)
+				(color 255 0 0 1)
+			)
+		)
+	)
 	(text "NOR flash memory 256 Mbit (32 MB x 8, 200 MHz)"
 		(exclude_from_sim no)
@@
 		)
 	)
+	(polyline
+		(pts
+			(xy 111.76 124.46) (xy 114.3 127)
+		)
+		(stroke
+			(width 0)
+			(type solid)
+			(color 255 0 0 1)
+		)
+	)
 	(wire
 		(pts
@@
 		)
 	)
+	(polyline
+		(pts
+			(xy 107.315 94.615) (xy 111.76 98.425)
+		)
+		(stroke
+			(width 0)
+			(type solid)
+			(color 255 0 0 1)
+		)
+	)
 	(wire
 		(pts
@@
 		)
 	)
+	(polyline
+		(pts
+			(xy 88.265 94.615) (xy 107.315 94.615)
+		)
+		(stroke
+			(width 0)
+			(type solid)
+			(color 255 0 0 1)
+		)
+	)
 	(wire
 		(pts
@@
 		)
 	)
+	(polyline
+		(pts
+			(xy 111.76 98.425) (xy 111.76 124.46)
+		)
+		(stroke
+			(width 0)
+			(type solid)
+			(color 255 0 0 1)
+		)
+	)

Commit message: #16
Parts:
- added JP1, JP2, JP3, JP4, JP5: ~, PCM_EEZ_SMD:JP3 shorted (0603), symbol PCM_EEZ_unsorted:JP3 shorted
- added R25, R30, R31: 10K, PCM_EEZ_passives:R_0402_1005Metric, symbol PCM_EEZ_passives:R-EU
- renumbered C76 to C63, C77 to C64, C78 to C65, C79 to C66, C80 to C67, C81 to C68, C63 to C69, C66 to C70, C68 to C71, C69 to C72, C64 to C73, C70 to C74, C74 to C75, C75 to C76, C65 to C77, C67 to C78, C71 to C79, C72 to C80, C73 to C81, IC12 to IC10, IC10 to IC11, IC11 to IC12, JP2 to JP6, R25 to R20, R28 to R21, R21 to R22, R22 to R23, R23 to R24, R24 to R26, R26 to R27, R27 to R28, R20 to R29
Connections:
- net +3V3: now also JP3.NO, JP5.NO, R31.2
- net GND: now also JP3.NC, JP5.NC, R25.2, R30.2; no longer IC9.10 (~{PD}), IC9.35 (DKEN), R23.2
- net SCL: now also JP2.NC; no longer IC9.15 (BSEL/SCL)
- net SDA: now also JP4.NC; no longer IC9.14 (DSEL/SDA)
- net TVDD: now also R23.2
- net ~{RESET_OUT}: now also JP1.NC; no longer IC9.13 (ISEL/~{RST})
- new net: IC9.13 (ISEL/~{RST}), JP1.COM
- new net: JP1.NO, R25.1
- new net: IC9.10 (~{PD}), JP3.COM
- new net: IC9.35 (DKEN), JP5.COM
- new net: IC9.14 (DSEL/SDA), JP4.COM
- new net: IC9.15 (BSEL/SCL), JP2.COM
- new net: JP4.NO, R31.1
- new net: JP2.NO, R30.1
Other:
- note removed: "Connect?"
- moved on the sheet: C63, C64, C65, C66, C67, C68, C69, C70, C71, C72, C73, C74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

Commit message: #17
Parts:
- added JP1: ~, PCM_EEZ_SMD:JP3 shorted (0603), symbol PCM_EEZ_unsorted:JP3 shorted
- R24: value 1K -> 10K; DigiKey 13-RC0402FR-131KLCT-ND -> 311-10.0KLRCT-ND; LCSC C4247997 -> C60490; Mouser 603-RC0402FR-131KL -> 603-RC0402FR-0710KL; TME SMD0402-1K-1% -> SMD0402-10K-1%; now not fitted; now left out of the parts list
- R29: value 4K7 -> 10K; DigiKey 13-RC0402FR-104K7LCT-ND -> 311-10.0KLRCT-ND; LCSC (none) -> C60490; Mouser 603-RC0402FR-104K7L -> 603-RC0402FR-0710KL; TME SMD0402-4K7-1% -> SMD0402-10K-1%
- renumbered JP1 to JP2, JP2 to JP3, JP3 to JP4, JP4 to JP5, JP5 to JP6, JP6 to JP7, R26 to R25, R25 to R26
Connections:
- net DVID_HPD: now also JP1.NC
- net at IC11.19 (HPD_A): now also R25.1
- net at IC11.21 (HPD_B), IC12.4 (A3): no longer R25.1
- net at R24.1: now also JP1.NO; no longer IC9.9 (EDGE/HTPLG)
- new net: IC9.9 (EDGE/HTPLG), JP1.COM
- no-connect marks 6 -> 5
Other:
- note removed: "Pulldown?"
- moved on the sheet: R25

Commit message: #18, OSHW ID121
Parts:
- C63, C65, C67, C69, C70, C71, C73, C75, C76, C77, C78, C81: LCSC (none) -> C60474
- C80: LCSC (none) -> C15195
- R23: LCSC (none) -> C276273
Changed lines of the file:
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@@
 	(title_block
 		(title "${project_name}")
-		(date "2026-04-01")
+		(date "2026-04-04")
 		(rev "${project_version}")
 		(company "${project_creator}")
@@
 			)
 		)
-		(property "LCSC" ""
+		(property "LCSC" "C60474"
 			(at 96.52 114.3 0)
 			(effects
@@
 			)
 		)
-		(property "LCSC" ""
+		(property "LCSC" "C60474"
 			(at 243.84 30.48 0)
 			(effects
@@
 			)
 		)
-		(property "LCSC" ""
+		(property "LCSC" "C60474"
 			(at 101.6 127 0)
 			(effects
@@
 			)
 		)
-		(property "LCSC" ""
+		(property "LCSC" "C60474"
 			(at 96.52 101.6 0)
 			(effects
@@
 			)
 		)
-		(property "LCSC" ""
+		(property "LCSC" "C60474"
 			(at 106.68 101.6 0)
 			(effects
@@
 			)
 		)
-		(property "LCSC" ""
+		(property "LCSC" "C276273"
 			(at 99.06 71.12 0)
 			(effects
@@
 		)
 		(instances
-			(project ""
+			(project "BB3plus CM5 STM32H7 module"
 				(path "/1a4f0aea-3a69-423f-8790-3103cd0321c4/6c545e17-ca5e-4b04-9dff-4169dbe59c9e"
 					(reference "IC12")
@@
 			)
 		)
-		(property "LCSC" ""
+		(property "LCSC" "C60474"
 			(at 101.6 101.6 0)
 			(effects
@@
 			)
 		)
-		(property "LCSC" ""
+		(property "LCSC" "C60474"
 			(at 210.82 116.84 0)
 			(effects
@@
 			)
 		)
-		(property "LCSC" ""
+		(property "LCSC" "C60474"
 			(at 256.54 30.48 0)
 			(effects
@@
 			)
 		)
-		(property "LCSC" ""
+		(property "LCSC" "C60474"
 			(at 246.38 116.84 0)
 			(effects
@@
 			)
 		)
-		(property "LCSC" ""
+		(property "LCSC" "C60474"
 			(at 96.52 127 0)
 			(effects
@@
 			)
 		)
-		(property "LCSC" ""
+		(property "LCSC" "C15195"
 			(at 193.04 139.7 0)
 			(effects
@@
 			)
 		)
-		(property "LCSC" ""
+		(property "LCSC" "C60474"
 			(at 198.12 139.7 0)
 			(effects
@@
 			)
 		)
-		(property "LCSC" ""
+		(property "LCSC" "C60474"
 			(at 231.14 30.48 0)
 			(effects

Commit message: #19
Parts:
- renumbered C63 to C58, C64 to C59, C65 to C60, C66 to C61, C67 to C62, C68 to C63, C69 to C64, C70 to C65, C71 to C66, C72 to C67, C73 to C68, C74 to C69, C75 to C70, C76 to C71, C77 to C72, C78 to C73, C79 to C74, C80 to C75, C81 to C76, IC11 to IC10, IC12 to IC11, IC9 to IC8, IC10 to IC9, R20 to R25, R21 to R26, R22 to R27, R23 to R28, R24 to R29, R25 to R30, R26 to R31, R27 to R32, R28 to R33, R29 to R34, R30 to R35, R31 to R36

Commit message: .step file update, migration to KiCad 10
Parts:
- JP1, JP2, JP3, JP4, JP5, JP6, JP7: value ~ -> (none)
