File: KiCad/Ethernet_flash.kicad_sch (KiCad schematic)
At the start: 45 parts, among them IC10 LSF0204GU12, IC11 MX25UM25645GXDI00-T, IC8 TFP410PAP, IC9 TS3DV642A0RUAR

Commit message: #24
Parts:
- added D1: BAT54XV2T5G, PCM_EEZ_SMD:SOD-523F_0P9X1P3_ONS, symbol PCM_EEZ_discretes:DIODE
- added R34: 10K, PCM_EEZ_passives:R_0402_1005Metric, symbol PCM_EEZ_passives:R-EU
- renumbered C73 to C72, C72 to C73, R34 to R35, R35 to R36, R36 to R37, R37 to R38
Connections:
- net +1V8: now also R34.2
- net ~{RESET_OUT}: now also D1.C; no longer IC11.A4 (~{RESET})
- new net 1V8_RST: D1.A, IC11.A4 (~{RESET}), R34.1
Other:
- moved on the sheet: C58, C59, C60, C61, C62, C63, C64, C65, C66, C67, C68, C69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
