File: KiCad/STM32H7_MCU.kicad_sch (KiCad schematic)
At the start: 49 parts, among them IC4 STM32H7R7L8H6H, IC5 SN74LVC1G14DBVR, Y1 VXM7-9032-25M0000000

Commit message: Split SoM footprint into two separate 100-pin connectors
Parts:
- renumbered C7 to C10, C12 to C11, C17 to C12, C8 to C13, C13 to C14, C19 to C15, C21 to C16, C9 to C17, C14 to C18, C22 to C19, C10 to C20, C15 to C21, C23 to C22, C26 to C23, C18 to C24, C11 to C25, C16 to C26, C24 to C27, C25 to C28, C30 to C29, C34 to C30, C42 to C31, C31 to C32, C35 to C33, C32 to C34, C37 to C35, C27 to C36, C33 to C37, C28 to C39, C39 to C40, C29 to C41, C40 to C42, C36 to C6, C41 to C7, C20 to C8, C6 to C9, IC5 to IC4, IC4 to IC5, R3 to R1, R4 to R2, R2 to R3, R1 to R4, X1 to X3

Commit message: Rename USB_FS_SEL to USB_HS_SEL
Connections:
- net USB_FS_SEL renamed USB_HS_SEL
Changed lines of the file:
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@@
 		)
 	)
-	(global_label "USB_FS_SEL"
+	(global_label "USB_HS_SEL"
 		(shape output)
 		(at 76.2 55.88 0)
@@
 		)
 		(property "Intersheetrefs" "${INTERSHEET_REFS}"
-			(at 85.8326 55.88 0)
+			(at 86.0019 55.88 0)
 			(hide yes)
 			(show_name no)

Commit message: #20
Parts:
- renumbered R1 to R2, R2 to R3, R3 to R4, R4 to R5
Changed lines of the file:
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@@
 	(title_block
 		(title "${project_name}")
-		(date "2026-04-18")
+		(date "2026-04-20")
 		(rev "${project_version}")
 		(company "${project_creator}")
@@
 		(in_pos_files yes)
 		(dnp no)
-		(property "Reference" "#PWR014"
+		(property "Reference" "#PWR015"
 			(at 251.46 80.01 0)
 			(hide yes)
@@
 			(project "BB3plus CM5 STM32H7 module"
 				(path "/1a4f0aea-3a69-423f-8790-3103cd0321c4/d7166dbe-caf3-45a8-82fe-1ff0a9696e25"
-					(reference "#PWR014")
+					(reference "#PWR015")
 					(unit 1)
 				)
@@
 		(in_pos_files yes)
 		(dnp no)
-		(property "Reference" "#+3V09"
+		(property "Reference" "#+3V010"
 			(at 185.42 99.06 0)
 			(hide yes)
@@
 			(project "BB3plus CM5 STM32H7 module"
 				(path "/1a4f0aea-3a69-423f-8790-3103cd0321c4/d7166dbe-caf3-45a8-82fe-1ff0a9696e25"
-					(reference "#+3V09")
+					(reference "#+3V010")
 					(unit 1)
 				)
@@
 		(in_pos_files yes)
 		(dnp no)
-		(property "Reference" "#PWR015"
+		(property "Reference" "#PWR016"
 			(at 270.51 109.22 0)
 			(hide yes)
@@
 			(project "BB3plus CM5 STM32H7 module"
 				(path "/1a4f0aea-3a69-423f-8790-3103cd0321c4/d7166dbe-caf3-45a8-82fe-1ff0a9696e25"
-					(reference "#PWR015")
+					(reference "#PWR016")
 					(unit 1)
 				)
@@
 		(in_pos_files yes)
 		(dnp no)
-		(property "Reference" "#+3V05"
+		(property "Reference" "#+3V06"
 			(at 22.86 170.18 0)
 			(hide yes)
@@
 			(project "BB3plus CM5 STM32H7 module"
 				(path "/1a4f0aea-3a69-423f-8790-3103cd0321c4/d7166dbe-caf3-45a8-82fe-1ff0a9696e25"
-					(reference "#+3V05")
+					(reference "#+3V06")
 					(unit 1)
 				)
@@
 		(in_pos_files yes)
 		(dnp no)
-		(property "Reference" "R3"
+		(property "Reference" "R4"
 			(at 157.48 74.93 90)
 			(show_name no)
@@
 			(project "BB3plus CM5 STM32H7 module"
 				(path "/1a4f0aea-3a69-423f-8790-3103cd0321c4/d7166dbe-caf3-45a8-82fe-1ff0a9696e25"
-					(reference "R3")
+					(reference "R4")
 					(unit 1)
 				)
@@
 		(in_pos_files yes)
 		(dnp no)
-		(property "Reference" "R4"
+		(property "Reference" "R5"
 			(at 171.45 61.595 0)
 			(show_name no)
@@
 			(project "BB3plus CM5 STM32H7 module"
 				(path "/1a4f0aea-3a69-423f-8790-3103cd0321c4/d7166dbe-caf3-45a8-82fe-1ff0a9696e25"
-					(reference "R4")
+					(reference "R5")
 					(unit 1)
 				)
@@
 		(in_pos_files yes)
 		(dnp no)
-		(property "Reference" "#+3V07"
+		(property "Reference" "#+3V08"
 			(at 175.26 50.8 0)
 			(hide yes)
@@
 			(project "BB3plus CM5 STM32H7 module"
 				(path "/1a4f0aea-3a69-423f-8790-3103cd0321c4/d7166dbe-caf3-45a8-82fe-1ff0a9696e25"
-					(reference "#+3V07")
+					(reference "#+3V08")
 					(unit 1)
 				)
@@
 		(in_pos_files yes)
 		(dnp no)
-		(property "Reference" "#PWR016"
+		(property "Reference" "#PWR017"
 			(at 273.05 132.08 0)
 			(hide yes)
@@
 			(project "BB3plus CM5 STM32H7 module"
 				(path "/1a4f0aea-3a69-423f-8790-3103cd0321c4/d7166dbe-caf3-45a8-82fe-1ff0a9696e25"
-					(reference "#PWR016")
+					(reference "#PWR017")
 					(unit 1)
 				)
@@
 		(in_pos_files yes)
 		(dnp no)
-		(property "Reference" "R1"
+		(property "Reference" "R2"
 			(at 90.17 105.41 0)
 			(show_name no)
@@
 			(project "BB3plus CM5 STM32H7 module"
 				(path "/1a4f0aea-3a69-423f-8790-3103cd0321c4/d7166dbe-caf3-45a8-82fe-1ff0a9696e25"
-					(reference "R1")
+					(reference "R2")
 					(unit 1)
 				)
@@
 		(in_pos_files yes)
 		(dnp no)
-		(property "Reference" "#+3V06"
+		(property "Reference" "#+3V07"
 			(at 93.98 100.33 0)
 			(hide yes)
@@
 			(project "BB3plus CM5 STM32H7 module"
 				(path "/1a4f0aea-3a69-423f-8790-3103cd0321c4/d7166dbe-caf3-45a8-82fe-1ff0a9696e25"
-					(reference "#+3V06")
+					(reference "#+3V07")
 					(unit 1)
 				)
@@
 		(in_pos_files yes)
 		(dnp no)
-		(property "Reference" "R2"
+		(property "Reference" "R3"
 			(at 95.25 105.41 0)
 			(show_name no)
@@
 			(project "BB3plus CM5 STM32H7 module"
 				(path "/1a4f0aea-3a69-423f-8790-3103cd0321c4/d7166dbe-caf3-45a8-82fe-1ff0a9696e25"
-					(reference "R2")
+					(reference "R3")
 					(unit 1)
 				)
@@
 		(dnp no)
 		(fields_autoplaced yes)
-		(property "Reference" "#+3V08"
+		(property "Reference" "#+3V09"
 			(at 177.8 27.94 0)
 			(hide yes)
@@
 			(project "BB3plus CM5 STM32H7 module"
 				(path "/1a4f0aea-3a69-423f-8790-3103cd0321c4/d7166dbe-caf3-45a8-82fe-1ff0a9696e25"
-					(reference "#+3V08")
+					(reference "#+3V09")
 					(unit 1)
 				)

Commit message: #21
Connections:
- net ~{ETH_RESET}: now reaches IC5.D1 (PC15-OSC32_O_UT)
- no-connect marks 26 -> 25
Changed lines of the file:
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@@
 	)
 	(no_connect
+		(at 40.64 91.44)
+	)
+	(no_connect
 		(at 71.12 38.1)
 	)
@@
 	)
 	(no_connect
-		(at 40.64 91.44)
-	)
-	(no_connect
 		(at 71.12 43.18)
 	)
@@
 		(at 119.38 58.42)
 	)
-	(no_connect
-		(at 40.64 152.4)
-	)
 	(bus_entry
 		(at 106.68 88.9)
@@
 	(wire
 		(pts
+			(xy 35.56 152.4) (xy 40.64 152.4)
+		)
+		(stroke
+			(width 0)
+			(type default)
+		)
+	)
+	(wire
+		(pts
 			(xy 187.96 45.72) (xy 193.04 45.72)
 		)
@@
 			)
 		)
+	)
+	(global_label "~{ETH_RESET}"
+		(shape output)
+		(at 35.56 152.4 180)
+		(fields_autoplaced yes)
+		(effects
+			(font
+				(size 0.889 0.889)
+				(color 204 102 0 1)
+			)
+			(justify right)
+		)
+		(property "Intersheetrefs" "${INTERSHEET_REFS}"
+			(at 26.8166 152.4 0)
+			(hide yes)
+			(show_name no)
+			(do_not_autoplace no)
+			(effects
+				(font
+					(size 1.27 1.27)
+				)
+				(justify right)
+			)
+		)

Commit message: #22
Connections:
- net ETH_CLK: now reaches IC5.E7 (PD6)
- no-connect marks 25 -> 24
Changed lines of the file:
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@@
 	)
 	(no_connect
-		(at 71.12 43.18)
-	)
-	(no_connect
 		(at 71.12 58.42)
 	)
@@
 	(wire
 		(pts
+			(xy 71.12 43.18) (xy 76.2 43.18)
+		)
+		(stroke
+			(width 0)
+			(type default)
+		)
+	)
+	(wire
+		(pts
 			(xy 210.82 99.06) (xy 210.82 106.68)
 		)
@@
 			)
 		)
+	)
+	(global_label "ETH_CLK"
+		(shape output)
+		(at 76.2 43.18 0)
+		(fields_autoplaced yes)
+		(effects
+			(font
+				(size 0.889 0.889)
+				(color 204 102 0 1)
+			)
+			(justify left)
+		)
+		(property "Intersheetrefs" "${INTERSHEET_REFS}"
+			(at 83.4195 43.18 0)
+			(hide yes)
+			(show_name no)
+			(do_not_autoplace no)
+			(effects
+				(font
+					(size 1.27 1.27)
+				)
+				(justify left)
+			)
+		)

Commit message: #23
Connections:
- net GND: now also IC5.L13 (PD15), IC5.N13 (PD12), IC5.P14 (PD13)
- no-connect marks 24 -> 21
Changed lines of the file:
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@@
 	(title_block
 		(title "${project_name}")
-		(date "2026-04-21")
+		(date "2026-05-01")
 		(rev "${project_version}")
 		(company "${project_creator}")
@@
 		)
 	)
+	(text_box "Module ID: 000"
+		(exclude_from_sim no)
+		(at 88.9 48.26 0)
+		(size 12.7 15.24)
+		(margins 0.9525 0.9525 0.9525 0.9525)
+		(stroke
+			(width 0)
+			(type solid)
+			(color 132 0 132 1)
+		)
+		(fill
+			(type none)
+		)
+		(effects
+			(font
+				(size 0.889 0.889)
+				(color 132 0 132 1)
+			)
+			(justify left top)
+		)
+	)
+	(junction
+		(at 91.44 53.34)
+		(diameter 0)
+		(color 0 0 0 0)
+	)
 	(junction
 		(at 193.04 86.36)
@@
 	)
 	(junction
+		(at 91.44 58.42)
+		(diameter 0)
+		(color 0 0 0 0)
+	)
+	(junction
 		(at 248.92 91.44)
 		(diameter 0)
@@
 	)
 	(no_connect
-		(at 71.12 53.34)
-	)
-	(no_connect
 		(at 40.64 129.54)
 	)
@@
 	)
 	(no_connect
-		(at 71.12 50.8)
-	)
-	(no_connect
 		(at 71.12 83.82)
 	)
@@
 	)
 	(no_connect
-		(at 71.12 58.42)
-	)
-	(no_connect
 		(at 119.38 58.42)
 	)
@@
 		)
 	)
+	(wire
+		(pts
+			(xy 71.12 50.8) (xy 91.44 50.8)
+		)
+		(stroke
+			(width 0)
+			(type default)
+		)
+	)
 	(polyline
 		(pts
@@
 	(wire
 		(pts
+			(xy 71.12 58.42) (xy 91.44 58.42)
+		)
+		(stroke
+			(width 0)
+			(type default)
+		)
+	)
+	(wire
+		(pts
 			(xy 248.92 43.18) (xy 248.92 45.72)
 		)
@@
 	(wire
 		(pts
+			(xy 91.44 53.34) (xy 91.44 58.42)
+		)
+		(stroke
+			(width 0)
+			(type default)
+		)
+	)
+	(wire
+		(pts
 			(xy 246.38 63.5) (xy 248.92 63.5)
 		)
@@
 	(wire
 		(pts
+			(xy 71.12 53.34) (xy 91.44 53.34)
+		)
+		(stroke
+			(width 0)
+			(type default)
+		)
+	)
+	(wire
+		(pts
 			(xy 248.92 96.52) (xy 248.92 99.06)
 		)
@@
 	(wire
 		(pts
+			(xy 91.44 50.8) (xy 91.44 53.34)
+		)
+		(stroke
+			(width 0)
+			(type default)
+		)
+	)
+	(wire
+		(pts
 			(xy 154.94 93.98) (xy 149.86 93.98)
 		)
@@
 					(unit 1)
 				)
+			)
+		)
+	)
+	(symbol
+		(lib_id "PCM_EEZ_symbols:GND")
+		(at 91.44 60.96 0)
+		(mirror y)
+		(unit 1)
+		(body_style 1)
+		(exclude_from_sim no)
+		(in_bom yes)
+		(on_board yes)
+		(in_pos_files yes)
+		(dnp no)
+		(property "Reference" "#SUPPLY053"
+			(at 91.44 60.96 0)
+			(hide yes)
+			(show_name no)
+			(do_not_autoplace no)
+			(effects
+				(font
+					(size 1.27 1.27)
+				)
+			)
+		)
+		(property "Value" "GND"
+			(at 93.345 62.23 0)
+			(show_name no)
+			(do_not_autoplace no)
+			(effects
+				(font
+					(size 1.27 1.27)
+				)
+				(justify right bottom)
+			)
+		)
+		(property "Footprint" ""
+			(at 91.44 60.96 0)
+			(hide yes)
+			(show_name no)
+			(do_not_autoplace no)
+			(effects
+				(font
+					(size 1.27 1.27)
+				)
+			)
+		)
+		(property "Datasheet" ""
+			(at 91.44 60.96 0)
+			(hide yes)
+			(show_name no)
+			(do_not_autoplace no)
+			(effects
+				(font
+					(size 1.27 1.27)
+				)
+			)
+		)
+		(property "Description" ""
+			(at 91.44 60.96 0)
+			(hide yes)
+			(show_name no)
+			(do_not_autoplace no)
+			(effects
+				(font
+					(size 1.27 1.27)
+				)
+			)
+		)
+		(pin "1"
+		)
+		(instances
+			(project "BB3plus CM5 STM32H7 module"
+				(path "/1a4f0aea-3a69-423f-8790-3103cd0321c4/d7166dbe-caf3-45a8-82fe-1ff0a9696e25"
+					(reference "#SUPPLY053")
+					(unit 1)
+				)
