File: KiCad/cm5_socket_mcu.kicad_sch (KiCad schematic)
At the start: 12 parts, among them IC1 AZ1117CH2-3.3TRG1, IC2 AZ1117CH-1.8TRG1, IC3 PI3USB102ZLEX, X1 DF40C-100DP-0.4V(51), X2 DF40C-100DP-0.4V(51)

Commit message: #25
Connections:
- net DIN2: now also X1.97 (CAM_GPIO0); no longer X1.35 (ID_SC/GPIO1)
- net RS485_RX/DIN3: now also X1.35 (ID_SC/GPIO1); no longer X1.100 (CAM_GPIO1)
- net RS485_TX/DOUT3: now also X1.36 (ID_SD/GPIO0); no longer X1.97 (CAM_GPIO0)
- net RTC_CM5: now also X1.100 (CAM_GPIO1); no longer X1.36 (ID_SD/GPIO0)
Changed lines of the file:
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@@
 	(title_block
 		(title "${project_name}")
-		(date "2026-07-10")
+		(date "2026-09-17")
 		(rev "${project_version}")
 		(company "${project_creator}")
@@
 	(wire
 		(pts
-			(xy 40.64 121.92) (xy 50.8 121.92)
+			(xy 43.18 121.92) (xy 50.8 121.92)
 		)
 		(stroke
@@
 	(wire
 		(pts
-			(xy 40.64 139.7) (xy 50.8 139.7)
+			(xy 43.18 139.7) (xy 50.8 139.7)
 		)
 		(stroke
@@
 		)
 	)
-	(wire
-		(pts
-			(xy 43.18 68.58) (xy 50.8 68.58)
-		)
-		(stroke
-			(width 0)
-			(type default)
-		)
-	)
 	(polyline
 		(pts
@@
 		)
 	)
+	(wire
+		(pts
+			(xy 109.22 147.32) (xy 101.6 147.32)
+		)
+		(stroke
+			(width 0)
+			(type default)
+		)
+	)
 	(polyline
 		(pts
@@
 	(wire
 		(pts
+			(xy 43.18 149.86) (xy 50.8 149.86)
+		)
+		(stroke
+			(width 0)
+			(type default)
+		)
+	)
+	(wire
+		(pts
 			(xy 147.32 139.7) (xy 149.86 139.7)
 		)
@@
 	(wire
 		(pts
-			(xy 40.64 149.86) (xy 50.8 149.86)
-		)
-		(stroke
-			(width 0)
-			(type default)
-		)
-	)
-	(wire
-		(pts
 			(xy 231.14 45.72) (xy 233.68 45.72)
 		)
@@
 		)
 	)
-	(wire
-		(pts
-			(xy 101.6 147.32) (xy 109.22 147.32)
-		)
-		(stroke
-			(width 0)
-			(type default)
-		)
-	)
 	(polyline
 		(pts
@@
 	(wire
 		(pts
-			(xy 40.64 124.46) (xy 50.8 124.46)
+			(xy 43.18 124.46) (xy 50.8 124.46)
 		)
 		(stroke
@@
 	(wire
 		(pts
+			(xy 43.18 68.58) (xy 50.8 68.58)
+		)
+		(stroke
+			(width 0)
+			(type default)
+		)
+	)
+	(wire
+		(pts
 			(xy 142.24 88.9) (xy 149.86 88.9)
 		)
@@
 	(wire
 		(pts
-			(xy 101.6 68.58) (xy 109.22 68.58)
-		)
-		(stroke
-			(width 0)
-			(type default)
-		)
-	)
-	(wire
-		(pts
 			(xy 45.72 134.62) (xy 50.8 134.62)
 		)
@@
 	(wire
 		(pts
-			(xy 40.64 127) (xy 50.8 127)
+			(xy 43.18 127) (xy 50.8 127)
 		)
 		(stroke
@@
 	(wire
 		(pts
+			(xy 109.22 68.58) (xy 101.6 68.58)
+		)
+		(stroke
+			(width 0)
+			(type default)
+		)
+	)
+	(wire
+		(pts
 			(xy 60.96 177.8) (xy 60.96 180.34)
 		)
@@
 	(global_label "SCL"
 		(shape bidirectional)
-		(at 40.64 124.46 180)
+		(at 43.18 124.46 180)
 		(fields_autoplaced yes)
 		(effects
@@
 		)
 		(property "Intersheetrefs" "${INTERSHEET_REFS}"
-			(at 35.8862 124.46 0)
+			(at 38.4262 124.46 0)
 			(hide yes)
 			(show_name no)
@@
 	(global_label "DIN2"
 		(shape output)
-		(at 109.22 68.58 0)
+		(at 109.22 147.32 0)
 		(fields_autoplaced yes)
 		(effects
@@
 		)
 		(property "Intersheetrefs" "${INTERSHEET_REFS}"
-			(at 113.9419 68.58 0)
+			(at 113.9419 147.32 0)
 			(hide yes)
 			(show_name no)
@@
 	(global_label "~{RESET_OUT}"
 		(shape output)
-		(at 40.64 139.7 180)
+		(at 43.18 139.7 180)
 		(fields_autoplaced yes)
 		(effects
@@
 		)
 		(property "Intersheetrefs" "${INTERSHEET_REFS}"
-			(at 31.7696 139.7 0)
+			(at 34.3096 139.7 0)
 			(hide yes)
 			(show_name no)
@@
 	(global_label "GPIO_VREF"
 		(shape output)
-		(at 40.64 121.92 180)
+		(at 43.18 121.92 180)
 		(fields_autoplaced yes)
 		(effects
@@
 		)
 		(property "Intersheetrefs" "${INTERSHEET_REFS}"
-			(at 31.9812 121.92 0)
+			(at 34.5212 121.92 0)
 			(hide yes)
 			(show_name no)
@@
 	(global_label "SDA"
 		(shape bidirectional)
-		(at 40.64 127 180)
+		(at 43.18 127 180)
 		(fields_autoplaced yes)
 		(effects
@@
 		)
 		(property "Intersheetrefs" "${INTERSHEET_REFS}"
-			(at 35.8439 127 0)
+			(at 38.3839 127 0)
 			(hide yes)
 			(show_name no)
@@
 	(global_label "RS485_RX{slash}DIN3"
 		(shape output)
-		(at 40.64 149.86 180)
+		(at 109.22 68.58 0)
 		(fields_autoplaced yes)
 		(effects
@@
 				(size 0.889 0.889)
 			)
-			(justify right)
+			(justify left)
 		)
 		(property "Intersheetrefs" "${INTERSHEET_REFS}"
-			(at 28.298 149.86 0)
+			(at 121.562 68.58 0)
 			(hide yes)
 			(show_name no)
@@
 					(size 1.27 1.27)
 				)
-				(justify right)
+				(justify left)
 			)
 		)
@@
 	(global_label "RS485_TX{slash}DOUT3"
 		(shape input)
-		(at 109.22 147.32 0)
+		(at 43.18 68.58 180)
 		(fields_autoplaced yes)
 		(effects
@@
 				(size 0.889 0.889)
 			)
-			(justify left)
+			(justify right)
 		)
 		(property "Intersheetrefs" "${INTERSHEET_REFS}"
-			(at 122.5356 147.32 0)
+			(at 29.8644 68.58 0)
 			(hide yes)
 			(show_name no)
@@
 					(size 1.27 1.27)
 				)
-				(justify left)
+				(justify right)
 			)
 		)
@@
 	(global_label "RTC_CM5"
 		(shape output)
-		(at 43.18 68.58 180)
+		(at 43.18 149.86 180)
 		(fields_autoplaced yes)
 		(effects
@@
 		)
 		(property "Intersheetrefs" "${INTERSHEET_REFS}"
-			(at 35.6641 68.58 0)
+			(at 35.6641 149.86 0)
 			(hide yes)
 			(show_name no)
@@
 					(reference "R1")
 					(unit 1)
-					(variant
-						(name "Ethernet PHY no xtal")
-					)
 				)
 			)
@@
 					(reference "IC1")
 					(unit 1)
-					(variant
-						(name "Ethernet PHY no xtal")
-					)
 				)
 			)
@@
 					(reference "C4")
 					(unit 1)
-					(variant
-						(name "Ethernet PHY no xtal")
-					)
 				)
 			)
@@
 					(reference "C5")
 					(unit 1)
-					(variant
-						(name "Ethernet PHY no xtal")
-					)
 				)
 			)
@@
 					(reference "C3")
 					(unit 1)
-					(variant
-						(name "Ethernet PHY no xtal")
-					)
 				)
 			)
@@
 					(reference "IC3")
 					(unit 1)
-					(variant
-						(name "Ethernet PHY no xtal")
-					)
 				)
 			)
@@
 					(reference "IC2")
 					(unit 1)
-					(variant
-						(name "Ethernet PHY no xtal")
-					)
 				)
 			)
@@
 					(reference "X1")
 					(unit 1)
-					(variant
-						(name "Ethernet PHY no xtal")
-					)
 				)
 			)
@@
 					(reference "C1")
 					(unit 1)
-					(variant
-						(name "Ethernet PHY no xtal")
-					)
 				)
 			)
@@
 					(reference "JP1")
 					(unit 1)
-					(variant
-						(name "Ethernet PHY no xtal")
-					)
 				)
 			)
@@
 					(reference "C2")
 					(unit 1)
-					(variant
-						(name "Ethernet PHY no xtal")
-					)
 				)
 			)
@@
 					(reference "X2")
 					(unit 1)
-					(variant
-						(name "Ethernet PHY no xtal")
-					)
 				)
 			)
